File: hardware/chispas.kicad_sch (KiCad schematic)
At the start: 47 parts, among them J2 Conn_01x04, J3 Conn_01x04, J4 Conn_01x06, J5 Conn_01x02, J6 TRAFO, U1 Heltec_WiFi_LoRa_32_V3, U2 PC817X2CSP9F, U3 PAM8302AASCR, U4 PEC11R-4230F-S0024

Commit message: PCB: pedido a LCSC hecho y combinado; R7 al CTR R09710NS (C18213426), el ALPS sin stock
Co-Authored-By: Claude Opus 5.5 <noreply@anthropic.com>
Parts:
- R7: LCSC Part C97444 -> C18213426; MPN RK097111080J -> R09710NS-FB15D7.0-B103-0044
Changed lines of the file:
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@@
 			)
 		)
-		(property "Datasheet" "https://lcsc.com/product-detail/Potentiometers-Variable-Resistors_ALPS_RK097111080J_RK097111080J_C97444.html"
+		(property "Datasheet" "https://www.lcsc.com/product-detail/C18213426.html"
 			(at 250.19 148.59 0)
 			(hide yes)
@@
 			)
 		)
-		(property "MPN" "RK097111080J"
+		(property "MPN" "R09710NS-FB15D7.0-B103-0044"
 			(at 250.19 153.67 0)
 			(hide yes)
@@
 			)
 		)
-		(property "LCSC Part" "C97444"
+		(property "LCSC Part" "C18213426"
 			(at 250.19 156.21 0)
 			(hide yes)

Commit message: PCB: R7 vuelve al potenciometro ALPS RK097111080J (C97444) en el esquema y la compra; el CTR solo para las 5 placas pedidas
Co-Authored-By: Claude Opus 5.5 <noreply@anthropic.com>
Parts:
- R7: LCSC Part C18213426 -> C97444; MPN R09710NS-FB15D7.0-B103-0044 -> RK097111080J
Changed lines of the file:
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@@
 			)
 		)
-		(property "Datasheet" "https://www.lcsc.com/product-detail/C18213426.html"
+		(property "Datasheet" "https://lcsc.com/product-detail/Potentiometers-Variable-Resistors_ALPS_RK097111080J_RK097111080J_C97444.html"
 			(at 250.19 148.59 0)
 			(hide yes)
@@
 			)
 		)
-		(property "MPN" "R09710NS-FB15D7.0-B103-0044"
+		(property "MPN" "RK097111080J"
 			(at 250.19 153.67 0)
 			(hide yes)
@@
 			)
 		)
-		(property "LCSC Part" "C18213426"
+		(property "LCSC Part" "C97444"
 			(at 250.19 156.21 0)
 			(hide yes)
